Commit message: Updated robot model to be compatible with ROS2. Fixed the robot arm to the world frame. Added launch files for rviz. Verified link transforms using joint state publisher gui

File: urdf/barista_robot.urdf.xacro (robot description, xacro)
@@ -1,8 +1,13 @@
-<?xml version="1.0" encoding="utf-8"?>
+<?xml version="1.0" ?>
 <!-- This URDF was automatically created by SolidWorks to URDF Exporter! Originally created by Stephen Brawner (brawner@gmail.com)
      Commit Version: 1.6.0-4-g7f85cfe  Build Version: 1.6.7995.38578
      For more information, please see http://wiki.ros.org/sw_urdf_exporter -->
 <robot
-  name="barista_robot">
+  name="barista_robot" xmlns:xacro="http://ros.org/wiki/xacro">
+  <link name="world" />
+  <joint name="fixed_base" type="fixed">
+      <parent link="world" />
+      <child link="base_link" />
+  </joint>
   <link
     name="base_link">
@@ -35,4 +40,5 @@
       </material>
     </visual>
+    <static>true</static>
     <collision>
       <origin
@@ -669,5 +675,5 @@
   </link>
   <joint
-    name="right_finger_2"
+    name="right_finger_2_joint"
     type="continuous">
     <origin

Commit message: Updated colors of the robot

File: urdf/barista_robot.urdf.xacro (robot description, xacro)
@@ -5,4 +5,24 @@
 <robot
   name="barista_robot" xmlns:xacro="http://ros.org/wiki/xacro">
+  <xacro:macro name="grey_color">
+      <visual>
+      <material>
+          <ambient>0.250980392156863 0.250980392156863 0.250980392156863 1</ambient>
+          <diffuse>0.250980392156863 0.250980392156863 0.250980392156863 1</diffuse>
+          <specular>0.1 0.1 0.1 1</specular>
+          <emissive>0 0 0 0</emissive>
+      </material>
+      </visual>
+  </xacro:macro>
+  <xacro:macro name="red_color">
+      <visual>
+      <material>
+          <ambient>1 0.501960784313725 0.501960784313725 1</ambient>
+          <diffuse> 0.501960784313725 0.501960784313725 1 </diffuse>
+          <specular>0.1 0.1 0.1 1</specular>
+          <emissive>0 0 0 0</emissive>
+      </material>
+      </visual>
+  </xacro:macro>
   <link name="world" />
   <joint name="fixed_base" type="fixed">
@@ -14,5 +34,5 @@
     <inertial>
       <origin
-        xyz="0.00383011072526205 0.457157273514301 -0.000928737788211971"
+        xyz="0.00383011072526205 0.000928737788211999 0.457157273514301"
         rpy="0 0 0" />
       <mass
@@ -20,9 +40,9 @@
       <inertia
         ixx="1.87464355002268"
-        ixy="-0.014715478905658"
-        ixz="2.53087124754718E-05"
-        iyy="0.11834660940371"
-        iyz="0.00356830501660723"
-        izz="1.87476517415076" />
+        ixy="-2.53087124754727E-05"
+        ixz="-0.014715478905658"
+        iyy="1.87476517415076"
+        iyz="-0.00356830501660734"
+        izz="0.11834660940371" />
     </inertial>
     <visual>
@@ -37,8 +57,7 @@
         name="">
         <color
-          rgba="0.792156862745098 0.819607843137255 0.933333333333333 1" />
-      </material>
-    </visual>
-    <static>true</static>
+          rgba="0.250980392156863 0.250980392156863 0.250980392156863 1" />
+      </material>
+    </visual>
     <collision>
       <origin
@@ -55,5 +74,5 @@
     <inertial>
       <origin
-        xyz="-8.25728228697759E-05 0.0620784408679793 -0.00108614239219215"
+        xyz="-8.25728228697777E-05 0.0620784408679793 -0.00108614239219215"
         rpy="0 0 0" />
       <mass
@@ -61,6 +80,6 @@
       <inertia
         ixx="0.0031562038651467"
-        ixy="-2.7668784170352E-06"
-        ixz="-8.66772096465901E-07"
+        ixy="-2.76687841703515E-06"
+        ixz="-8.66772096465886E-07"
         iyy="0.00496373152249205"
         iyz="-5.19354690470229E-05"
@@ -78,5 +97,5 @@
         name="">
         <color
-          rgba="0.792156862745098 0.819607843137255 0.933333333333333 1" />
+          rgba="1 0.501960784313725 0.501960784313725 1" />
       </material>
     </visual>
@@ -93,8 +112,8 @@
   <joint
     name="robot_base_joint"
-    type="continuous">
-    <origin
-      xyz="0.00764723572178816 0.00185432675440543 0.912764586526285"
-      rpy="1.56875557980304 0.00837565350850774 -0.00110679099009043" />
+    type="fixed">
+    <origin
+      xyz="0.0076472 0.0018543 0.91276"
+      rpy="1.5688 0.0083757 -0.0011068" />
     <parent
       link="base_link" />
@@ -102,11 +121,11 @@
       link="robot_base" />
     <axis
-      xyz="0 1 0" />
-  </joint>
-  <link
-    name="Link_1">
-    <inertial>
-      <origin
-        xyz="5.29382164110885E-08 0.0850432466695747 0.0128932752104662"
+      xyz="0 0 0" />
+  </joint>
+  <link
+    name="link_1">
+    <inertial>
+      <origin
+        xyz="5.29382164128232E-08 0.0850432466695747 0.0128932752104662"
         rpy="0 0 0" />
       <mass
@@ -114,6 +133,6 @@
       <inertia
         ixx="0.0144417466716968"
-        ixy="-1.76720854918966E-07"
-        ixz="1.27033528348874E-07"
+        ixy="-1.76720854918668E-07"
+        ixz="1.27033528349741E-07"
         iyy="0.0120175511780906"
         iyz="-0.000178584855651563"
@@ -126,19 +145,19 @@
       <geometry>
         <mesh
-          filename="package://barista_robot/meshes/Link_1.STL" />
-      </geometry>
-      <material
-        name="">
-        <color
-          rgba="0.792156862745098 0.819607843137255 0.933333333333333 1" />
-      </material>
-    </visual>
-    <collision>
-      <origin
-        xyz="0 0 0"
-        rpy="0 0 0" />
-      <geometry>
-        <mesh
-          filename="package://barista_robot/meshes/Link_1.STL" />
+          filename="package://barista_robot/meshes/link_1.STL" />
+      </geometry>
+      <material
+        name="">
+        <color
+          rgba="1 0.501960784313725 0.501960784313725 1" />
+      </material>
+    </visual>
+    <collision>
+      <origin
+        xyz="0 0 0"
+        rpy="0 0 0" />
+      <geometry>
+        <mesh
+          filename="package://barista_robot/meshes/link_1.STL" />
       </geometry>
     </collision>
@@ -146,14 +165,19 @@
   <joint
     name="link_1_joint"
-    type="continuous">
-    <origin
-      xyz="0 0.0992470344686496 0"
-      rpy="0 0.465852120972895 0" />
+    type="revolute">
+    <origin
+      xyz="0 0.099247 0"
+      rpy="0 0.46585 0" />
     <parent
       link="robot_base" />
     <child
-      link="Link_1" />
+      link="link_1" />
     <axis
       xyz="0 1 0" />
+    <limit
+      lower="-3.14"
+      upper="3.14"
+      effort="100"
+      velocity="3.14" />
   </joint>
   <link
@@ -161,15 +185,15 @@
     <inertial>
       <origin
-        xyz="-1.63538959695349E-06 0.211231437313278 0.152882713422171"
-        rpy="0 0 0" />
-      <mass
-        value="5.85231057682878" />
-      <inertia
-        ixx="0.421785968335089"
-        ixy="-4.66685653188514E-06"
-        ixz="-8.61905289833986E-07"
-        iyy="0.0183913104483783"
-        iyz="0.000922257532907184"
-        izz="0.418871238551212" />
+        xyz="-1.63530545009734E-06 0.211231437364917 0.152882713335174"
+        rpy="0 0 0" />
+      <mass
+        value="5.85231057454819" />
+      <inertia
+        ixx="0.421785968792057"
+        ixy="-4.66698955952136E-06"
+        ixz="-8.61933981188834E-07"
+        iyy="0.0183913103922809"
+        iyz="0.000922257685442064"
+        izz="0.418871238998585" />
     </inertial>
     <visual>
@@ -184,5 +208,5 @@
         name="">
         <color
-          rgba="0.792156862745098 0.819607843137255 0.933333333333333 1" />
+          rgba="1 0.501960784313725 0.501960784313725 1" />
       </material>
     </visual>
@@ -199,14 +223,19 @@
   <joint
     name="link_2_joint"
-    type="continuous">
-    <origin
-      xyz="0 0.0830544613923512 0.0241087363932672"
+    type="revolute">
+    <origin
+      xyz="0 0.083054 0.024109"
       rpy="0 0 0" />
     <parent
-      link="Link_1" />
+      link="link_1" />
     <child
       link="link_2" />
     <axis
       xyz="0 0 1" />
+    <limit
+      lower="-3.14"
+      upper="3.14"
+      effort="100"
+      velocity="3.14" />
   </joint>
   <link
@@ -214,15 +243,15 @@
     <inertial>
       <origin
-        xyz="1.53109355368816E-06 0.265809569731614 0.0201295876103251"
-        rpy="0 0 0" />
-      <mass
-        value="4.62234527435744" />
-      <inertia
-        ixx="0.198422158289813"
-        ixy="4.85999774938072E-06"
-        ixz="-1.51825927212357E-07"
-        iyy="0.00626605018267435"
-        iyz="0.00588106796982974"
-        izz="0.197534306912721" />
+        xyz="1.53110060815975E-06 0.265809569671053 0.0201295876152247"
+        rpy="0 0 0" />
+      <mass
+        value="4.62234527371938" />
+      <inertia
+        ixx="0.198422158428495"
+        ixy="4.85995234595538E-06"
+        ixz="-1.51823787104821E-07"
+        iyy="0.00626605018851334"
+        iyz="0.00588106797289478"
+        izz="0.197534307061617" />
     </inertial>
     <visual>
@@ -237,5 +266,5 @@
         name="">
         <color
-          rgba="0.792156862745098 0.819607843137255 0.933333333333333 1" />
+          rgba="1 0.501960784313725 0.501960784313725 1" />
       </material>
     </visual>
@@ -252,5 +281,5 @@
   <joint
     name="link_3_joint"
-    type="continuous">
+    type="revolute">
     <origin
       xyz="0 0.6126 0"
@@ -262,4 +291,9 @@
     <axis
       xyz="0 0 1" />
+    <limit
+      lower="-3.14"
+      upper="3.14"
+      effort="100"
+      velocity="3.14" />
   </joint>
   <link
@@ -267,15 +301,15 @@
     <inertial>
       <origin
-        xyz="-1.65259348634903E-06 0.00153989303001056 0.134078404594346"
-        rpy="0 0 0" />
-      <mass
-        value="0.952055695094421" />
-      <inertia
-        ixx="0.00181788273241634"
-        ixy="1.83047467793671E-08"
-        ixz="-2.83696234279008E-08"
-        iyy="0.00150425784631242"
-        iyz="-4.60370789807922E-05"
-        izz="0.00132306977062697" />
+        xyz="-1.65409067374393E-06 0.00153987297982727 0.134078386407816"
+        rpy="0 0 0" />
+      <mass
+        value="0.952056234394498" />
+      <inertia
+        ixx="0.00181788273252644"
+        ixy="1.83030713911664E-08"
+        ixz="-2.83699805857262E-08"
+        iyy="0.00150425784838232"
+        iyz="-4.60370793799838E-05"
+        izz="0.00132306977239992" />
     </inertial>
     <visual>
@@ -290,5 +324,5 @@
         name="">
         <color
-          rgba="0.792156862745098 0.819607843137255 0.933333333333333 1" />
+          rgba="1 0.501960784313725 0.501960784313725 1" />
       </material>
     </visual>
@@ -305,7 +339,7 @@
   <joint
     name="link_4_joint"
-    type="continuous">
-    <origin
-      xyz="0 0.571549999999962 0"
+    type="revolute">
+    <origin
+      xyz="0 0.57155 0"
       rpy="0 0 0" />
     <parent
@@ -315,4 +349,9 @@
     <axis
       xyz="0 0 1" />
+    <limit
+      lower="-3.14"
+      upper="3.14"
+      effort="100"
+      velocity="3.14" />
   </joint>
   <link
@@ -320,15 +359,15 @@
     <inertial>
       <origin
-        xyz="1.34223381187404E-07 0.107894808228803 0.00172519954497102"
-        rpy="0 0 0" />
-      <mass
-        value="0.852888053030417" />
-      <inertia
-        ixx="0.00143476123836806"
-        ixy="-5.45972664424141E-09"
-        ixz="4.83376041369174E-10"
-        iyy="0.00122172828134366"
-        iyz="-3.6765369527715E-05"
-        izz="0.00112162872969263" />
+        xyz="1.19754439253938E-07 0.107894811323263 0.00172520348120131"
+        rpy="0 0 0" />
+      <mass
+        value="0.852888399213539" />
+      <inertia
+        ixx="0.00143476123567499"
+        ixy="-5.38094070829317E-09"
+        ixz="4.87203904200569E-10"
+        iyy="0.00122172827947616"
+        iyz="-3.67653414285888E-05"
+        izz="0.00112162874820744" />
     </inertial>
     <visual>
@@ -343,5 +382,5 @@
         name="">
         <color
-          rgba="0.792156862745098 0.819607843137255 0.933333333333333 1" />
+          rgba="1 0.501960784313725 0.501960784313725 1" />
       </material>
     </visual>
@@ -358,7 +397,7 @@
   <joint
     name="link_5_joint"
-    type="continuous">
-    <origin
-      xyz="0 0.00233145785499556 0.150041263606732"
+    type="revolute">
+    <origin
+      xyz="0 0.0023315 0.15004"
       rpy="0 0 0" />
     <parent
@@ -368,4 +407,9 @@
     <axis
       xyz="0 1 0" />
+    <limit
+      lower="-3.14"
+      upper="3.14"
+      effort="100"
+      velocity="3.14" />
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
Commit message: Added  joint controllers, so robot does not collaspe on itself. Still need to develop actual controllers to move links.

File: urdf/barista_robot.urdf.xacro (robot description, xacro)
@@ -809,4 +809,63 @@
       xyz="0 0 0" />
   </joint>
+ <ros2_control name="GazeboSystem" type="system">
+ <hardware>
+     <plugin>gazebo_ros2_control/GazeboSystem</plugin>
+ </hardware>
+# Position Controller
+ <joint name="link_1_joint">
+     <command_interface name="position">
+         <param name="min">-3.14</param>
+         <param name="max">3.14</param>
+     </command_interface>
+     <state_interface name="position"/>
+     <state_interface name="velocity"/>
+ </joint>
+ <joint name="link_2_joint">
+     <command_interface name="position">
+         <param name="min">-3.14</param>
+         <param name="max">3.14</param>
+     </command_interface>
+     <state_interface name="position"/>
+     <state_interface name="velocity"/>
+ </joint>
+ <joint name="link_3_joint">
+     <command_interface name="position">
+         <param name="min">-3.14</param>
+         <param name="max">3.14</param>
+     </command_interface>
+     <state_interface name="position"/>
+     <state_interface name="velocity"/>
+ </joint>
+ <joint name="link_4_joint">
+     <command_interface name="position">
+         <param name="min">-3.14</param>
+         <param name="max">3.14</param>
+     </command_interface>
+     <state_interface name="position"/>
+     <state_interface name="velocity"/>
+ </joint>
+ <joint name="link_5_joint">
+     <command_interface name="position">
+         <param name="min">-3.14</param>
+         <param name="max">3.14</param>
+     </command_interface>
+     <state_interface name="position"/>
+     <state_interface name="velocity"/>
+ </joint>
+ <joint name="link_6_joint">
+     <command_interface name="position">
+         <param name="min">-3.14</param>
+         <param name="max">3.14</param>
+     </command_interface>
+     <state_interface name="position"/>
+     <state_interface name="velocity"/>
+ </joint>
+ </ros2_control>
+  <gazebo>
+      <plugin filename="libgazebo_ros2_control.so" name="gazebo_ros2_control">
+          <parameters>$(find barista_robot)/config/control.yaml</parameters>
+      </plugin>
+  </gazebo>
   <gazebo reference="base_link">
     <xacro:grey_color />

Commit message: Added controller to move robot joints to specific position. MAde custom world

File: urdf/barista_robot.urdf.xacro (robot description, xacro)
@@ -178,5 +178,5 @@
       lower="-3.14"
       upper="3.14"
-      effort="100"
+      effort="1000"
       velocity="3.14" />
   </joint>
@@ -236,5 +236,5 @@
       lower="-3.14"
       upper="3.14"
-      effort="100"
+      effort="1000"
       velocity="3.14" />
   </joint>
@@ -294,5 +294,5 @@
       lower="-3.14"
       upper="3.14"
-      effort="100"
+      effort="1000"
       velocity="3.14" />
   </joint>
@@ -352,5 +352,5 @@
       lower="-3.14"
       upper="3.14"
-      effort="100"
+      effort="1000"
       velocity="3.14" />
   </joint>
@@ -410,5 +410,5 @@
       lower="-3.14"
       upper="3.14"
-      effort="100"
+      effort="1000"
       velocity="3.14" />
   </joint>
@@ -468,5 +468,5 @@
       lower="-3.14"
       upper="3.14"
-      effort="100"
+      effort="1000"
       velocity="3.14" />
   </joint>
@@ -579,5 +579,5 @@
       lower="-3.14"
       upper="3.14"
-      effort="100"
+      effort="1000"
       velocity="3.14" />
   </joint>
@@ -637,5 +637,5 @@
       lower="-3.14"
       upper="3.14"
-      effort="100"
+      effort="1000"
       velocity="3.14" />
   </joint>
@@ -695,5 +695,5 @@
       lower="-3.14"
       upper="3.14"
-      effort="100"
+      effort="1000"
       velocity="3.14" />
   </joint>
@@ -753,5 +753,5 @@
       lower="-3.14"
       upper="3.14"
-      effort="100"
+      effort="1000"
       velocity="3.14" />
   </joint>
@@ -862,4 +862,36 @@
      <state_interface name="velocity"/>
  </joint>
+  <joint name="left_finger_1_joint">
+     <command_interface name="position">
+         <param name="min">-3.14</param>
+         <param name="max">3.14</param>
+     </command_interface>
+     <state_interface name="position"/>
+     <state_interface name="velocity"/>
+ </joint>
+  <joint name="left_finger_2_joint">
+     <command_interface name="position">
+         <param name="min">-3.14</param>
+         <param name="max">3.14</param>
+     </command_interface>
+     <state_interface name="position"/>
+     <state_interface name="velocity"/>
+ </joint>
+   <joint name="right_finger_1_joint">
+     <command_interface name="position">
+         <param name="min">-3.14</param>
+         <param name="max">3.14</param>
+     </command_interface>
+     <state_interface name="position"/>
+     <state_interface name="velocity"/>
+ </joint>
+  <joint name="right_finger_2_joint">
+     <command_interface name="position">
+         <param name="min">-3.14</param>
+         <param name="max">3.14</param>
+     </command_interface>
+     <state_interface name="position"/>
+     <state_interface name="velocity"/>
+ </joint>
  </ros2_control>
   <gazebo>

Commit message: Saving Progress

File: urdf/barista_robot.urdf.xacro (robot description, xacro)
@@ -814,52 +814,4 @@
  </hardware>
 # Position Controller
- <joint name="link_1_joint">
-     <command_interface name="position">
-         <param name="min">-3.14</param>
-         <param name="max">3.14</param>
-     </command_interface>
-     <state_interface name="position"/>
-     <state_interface name="velocity"/>
- </joint>
- <joint name="link_2_joint">
-     <command_interface name="position">
-         <param name="min">-3.14</param>
-         <param name="max">3.14</param>
-     </command_interface>
-     <state_interface name="position"/>
-     <state_interface name="velocity"/>
- </joint>
- <joint name="link_3_joint">
-     <command_interface name="position">
-         <param name="min">-3.14</param>
-         <param name="max">3.14</param>
-     </command_interface>
-     <state_interface name="position"/>
-     <state_interface name="velocity"/>
- </joint>
- <joint name="link_4_joint">
-     <command_interface name="position">
-         <param name="min">-3.14</param>
-         <param name="max">3.14</param>
-     </command_interface>
-     <state_interface name="position"/>
-     <state_interface name="velocity"/>
- </joint>
- <joint name="link_5_joint">
-     <command_interface name="position">
-         <param name="min">-3.14</param>
-         <param name="max">3.14</param>
-     </command_interface>
-     <state_interface name="position"/>
-     <state_interface name="velocity"/>
- </joint>
- <joint name="link_6_joint">
-     <command_interface name="position">
-         <param name="min">-3.14</param>
-         <param name="max">3.14</param>
-     </command_interface>
-     <state_interface name="position"/>
-     <state_interface name="velocity"/>
- </joint>
   <joint name="left_finger_1_joint">
      <command_interface name="position">
@@ -894,4 +846,53 @@
      <state_interface name="velocity"/>
  </joint>
+ #Velocity Controllers
+  <joint name="link_1_joint">
+     <command_interface name="velocity">
+         <param name="min">-10.0</param>
+         <param name="max">10.0</param>
+     </command_interface>
+     <state_interface name="position"/>
+     <state_interface name="velocity"/>
+ </joint>
+  <joint name="link_2_joint">
+     <command_interface name="velocity">
+         <param name="min">-10.0</param>
+         <param name="max">10.0</param>
+     </command_interface>
+     <state_interface name="position"/>
+     <state_interface name="velocity"/>
+ </joint>
+   <joint name="link_3_joint">
+     <command_interface name="velocity">
+         <param name="min">-10.0</param>
+         <param name="max">10.0</param>
+     </command_interface>
+     <state_interface name="position"/>
+     <state_interface name="velocity"/>
+ </joint>
+  <joint name="link_4_joint">
+     <command_interface name="velocity">
+         <param name="min">-10.0</param>
+         <param name="max">10.0</param>
+     </command_interface>
+     <state_interface name="position"/>
+     <state_interface name="velocity"/>
+ </joint>
+   <joint name="link_5_joint">
+     <command_interface name="velocity">
+         <param name="min">-10.0</param>
+         <param name="max">10.0</param>
+     </command_interface>
+     <state_interface name="position"/>
+     <state_interface name="velocity"/>
+ </joint>
+   <joint name="link_6_joint">
+     <command_interface name="velocity">
+         <param name="min">-10.0</param>
+         <param name="max">10.0</param>
+     </command_interface>
+     <state_interface name="position"/>
+     <state_interface name="velocity"/>
+ </joint>
  </ros2_control>
   <gazebo>
