Commit message: Saving Progress. Adding Effort Controller to compensate for gravity of links in simulation

File: urdf/barista_robot.urdf.xacro (robot description, xacro)
@@ -178,5 +178,5 @@
       lower="-3.14"
       upper="3.14"
-      effort="1000"
+      effort="100.0"
       velocity="3.14" />
   </joint>
@@ -236,5 +236,5 @@
       lower="-3.14"
       upper="3.14"
-      effort="1000"
+      effort="100.0"
       velocity="3.14" />
   </joint>
@@ -294,5 +294,5 @@
       lower="-3.14"
       upper="3.14"
-      effort="1000"
+      effort="100.0"
       velocity="3.14" />
   </joint>
@@ -352,5 +352,5 @@
       lower="-3.14"
       upper="3.14"
-      effort="1000"
+      effort="100.0"
       velocity="3.14" />
   </joint>
@@ -410,5 +410,5 @@
       lower="-3.14"
       upper="3.14"
-      effort="1000"
+      effort="100.0"
       velocity="3.14" />
   </joint>
@@ -468,5 +468,5 @@
       lower="-3.14"
       upper="3.14"
-      effort="1000"
+      effort="100.0"
       velocity="3.14" />
   </joint>
@@ -531,5 +531,5 @@
         rpy="0 0 0" />
       <mass
-        value="0.0276813354629505" />
+        value="0.001" />
       <inertia
         ixx="6.64066668853769E-06"
@@ -579,5 +579,5 @@
       lower="-3.14"
       upper="3.14"
-      effort="1000"
+      effort="100.0"
       velocity="3.14" />
   </joint>
@@ -589,5 +589,5 @@
         rpy="0 0 0" />
       <mass
-        value="0.00758717719600194" />
+        value="0.001" />
       <inertia
         ixx="2.6334781516959E-07"
@@ -637,5 +637,5 @@
       lower="-3.14"
       upper="3.14"
-      effort="1000"
+      effort="100.0"
       velocity="3.14" />
   </joint>
@@ -647,5 +647,5 @@
         rpy="0 0 0" />
       <mass
-        value="0.0276813354629504" />
+        value="0.001" />
       <inertia
         ixx="6.64066668853769E-06"
@@ -695,5 +695,5 @@
       lower="-3.14"
       upper="3.14"
-      effort="1000"
+      effort="100.0"
       velocity="3.14" />
   </joint>
@@ -705,5 +705,5 @@
         rpy="0 0 0" />
       <mass
-        value="0.00758717719600175" />
+        value="0.001" />
       <inertia
         ixx="2.6334781516958E-07"
@@ -753,5 +753,5 @@
       lower="-3.14"
       upper="3.14"
-      effort="1000"
+      effort="100.0"
       velocity="3.14" />
   </joint>
@@ -763,5 +763,5 @@
         rpy="0 0 0" />
       <mass
-        value="0.00456870619569645" />
+        value="0.001" />
       <inertia
         ixx="1.29743486402871E-07"
@@ -813,7 +813,7 @@
      <plugin>gazebo_ros2_control/GazeboSystem</plugin>
  </hardware>
-# Position Controller
+ # Velocity Controller
   <joint name="left_finger_1_joint">
-     <command_interface name="position">
+     <command_interface name="velocity">
          <param name="min">-3.14</param>
          <param name="max">3.14</param>
@@ -823,5 +823,5 @@
  </joint>
   <joint name="left_finger_2_joint">
-     <command_interface name="position">
+     <command_interface name="velocity">
          <param name="min">-3.14</param>
          <param name="max">3.14</param>
@@ -831,5 +831,5 @@
  </joint>
    <joint name="right_finger_1_joint">
-     <command_interface name="position">
+     <command_interface name="velocity">
          <param name="min">-3.14</param>
          <param name="max">3.14</param>
@@ -839,5 +839,5 @@
  </joint>
   <joint name="right_finger_2_joint">
-     <command_interface name="position">
+     <command_interface name="velocity">
          <param name="min">-3.14</param>
          <param name="max">3.14</param>
@@ -895,4 +895,95 @@
      <state_interface name="velocity"/>
  </joint>
+ # Effort Controllers
+   <joint name="link_1_joint">
+     <command_interface name="effort">
+         <param name="min">0.0</param>
+         <param name="max">100.0</param>
+     </command_interface>
+     <state_interface name="position"/>
+     <state_interface name="velocity"/>
+     <state_interface name="effort"/>
+ </joint>
+   <joint name="link_2_joint">
+     <command_interface name="effort">
+         <param name="min">0.0</param>
+         <param name="max">100.0</param>
+     </command_interface>
+     <state_interface name="position"/>
+     <state_interface name="velocity"/>
+     <state_interface name="effort"/>
+ </joint>
+    <joint name="link_3_joint">
+     <command_interface name="effort">
+         <param name="min">0.0</param>
+         <param name="max">100.0</param>
+     </command_interface>
+     <state_interface name="position"/>
+     <state_interface name="velocity"/>
+     <state_interface name="effort"/>
+ </joint>
+    <joint name="link_4_joint">
+     <command_interface name="effort">
+         <param name="min">0.0</param>
+         <param name="max">100.0</param>
+     </command_interface>
+     <state_interface name="position"/>
+     <state_interface name="velocity"/>
+     <state_interface name="effort"/>
+ </joint>
+    <joint name="link_5_joint">
+     <command_interface name="effort">
+         <param name="min">0.0</param>
+         <param name="max">100.0</param>
+     </command_interface>
+     <state_interface name="position"/>
+     <state_interface name="velocity"/>
+     <state_interface name="effort"/>
+ </joint>
+    <joint name="link_6_joint">
+     <command_interface name="effort">
+         <param name="min">0.0</param>
+         <param name="max">100.0</param>
+     </command_interface>
+     <state_interface name="position"/>
+     <state_interface name="velocity"/>
+     <state_interface name="effort"/>
+ </joint>
+    <joint name="left_finger_1_joint">
+     <command_interface name="effort">
+         <param name="min">0.0</param>
+         <param name="max">100.0</param>
+     </command_interface>
+     <state_interface name="position"/>
+     <state_interface name="velocity"/>
+     <state_interface name="effort"/>
+ </joint>
+     <joint name="left_finger_2_joint">
+     <command_interface name="effort">
+         <param name="min">0.0</param>
+         <param name="max">100.0</param>
+     </command_interface>
+     <state_interface name="position"/>
+     <state_interface name="velocity"/>
+     <state_interface name="effort"/>
+ </joint>
+     <joint name="right_finger_1_joint">
+     <command_interface name="effort">
+         <param name="min">0.0</param>
+         <param name="max">100.0</param>
+     </command_interface>
+     <state_interface name="position"/>
+     <state_interface name="velocity"/>
+     <state_interface name="effort"/>
+ </joint>
+     <joint name="right_finger_2_joint">
+     <command_interface name="effort">
+         <param name="min">0.0</param>
+         <param name="max">100.0</param>
+     </command_interface>
+     <state_interface name="position"/>
+     <state_interface name="velocity"/>
+     <state_interface name="effort"/>
+ </joint>
  </ros2_control>
   <gazebo>
