Commit message: made new world

File: worlds/coffee_machine_model/Coffee__machine_assy.urdf (robot description, URDF)
Before this commit: robot coffee_cup_with_rim_assy, 1 links, 0 joints
Links:
- link base_link: mass 0.141210670413946 -> 196.780003604201; geometry collision mesh filename=package://Coffee__machine_assy/meshes/base_link.STL; visual mesh filename=package://Coffee__machine_assy/meshes/base_link.STL
